Commit message: Add Room 315 Staubli gripper manipulation demo

File: mfja_staubli_manipulation_demos/hpp/room315_payload_box.urdf (robot description, URDF)
Before this commit: robot room315_payload_box, 1 links, 0 joints
Links:
- link base_link: geometry collision box size=0.07 0.05 0.06; visual box size=0.07 0.05 0.06

File: mfja_staubli_manipulation_demos/urdf/staubli_tx2_60l_gripper.urdf (robot description, URDF)
Before this commit: robot staubli_tx2_60l_suction, 13 links, 12 joints
Links:
- removed link suction_cup
- removed link suction_mount
- removed link suction_tcp
- added link gripper_base; collision box size=0.09 0.17 0.03; visual box size=0.09 0.17 0.03
- added link gripper_left_finger; collision box size=0.024 0.012 0.09; visual box size=0.024 0.012 0.09
- added link gripper_right_finger; collision box size=0.024 0.012 0.09; visual box size=0.024 0.012 0.09
- added link gripper_tcp
Joints:
- removed joint suction_cup_tcp
- removed joint suction_mount_cup
- removed joint tool0_suction_mount
- added joint gripper_base_left_finger: type fixed, parent gripper_base, child gripper_left_finger, origin xyz=0 0.075 0.045 rpy=0 0 0
- added joint gripper_base_right_finger: type fixed, parent gripper_base, child gripper_right_finger, origin xyz=0 -0.075 0.045 rpy=0 0 0
- added joint gripper_base_tcp: type fixed, parent gripper_base, child gripper_tcp, origin xyz=0 0 0.060 rpy=0 0 0
- added joint tool0_gripper_base: type fixed, parent tool0, child gripper_base, origin xyz=0 0 0.035 rpy=0 0 0
