Commit message: [description] Update gear models for the two-piece HPP tutorial

File: mfja_3rd_floor_description/urdf/gear_42.urdf (robot description, URDF)
Before this commit: robot gear_42, 1 links, 0 joints
Links:
- link base_link: geometry collision cylinder length=0.012 radius=0.021; collision cylinder length=0.014 radius=0.0075

File: mfja_3rd_floor_description/urdf/gear_plate.urdf (robot description, URDF)
Before this commit: robot gear_plate, 1 links, 0 joints
Links:
- link base_link: geometry collision box size=.01 .18 0.03; collision box size=.01 .18 0.03

File: mfja_3rd_floor_description/urdf/gear_support.urdf (robot description, URDF)
Before this commit: robot gear_support, 1 links, 0 joints
Links:
- link base_link: geometry collision box size=.004 .019 .162; collision box size=.004 .019 .162

Commit message: [description] Use stl file for visual models of gear 42.

File: mfja_3rd_floor_description/urdf/gear_42.urdf (robot description, URDF)
Before this commit: robot gear_42, 1 links, 0 joints
Links:
- link base_link: geometry collision cylinder length=0.012 radius=0.021; collision cylinder length=0.014 radius=0.0075
