Commit message: [description] Add two beams above Staubli robot.

File: mfja_3rd_floor_description/urdf/room315_environment.urdf (robot description, URDF)
Before this commit: robot room315_environment, 24 links, 23 joints
Links:
- added link room312_two_beams_above_staubli; collision box size=0.06 1.00 0.06; collision box size=0.06 1.00 0.06
Joints:
- added joint room312_two_beams_above_staubli_joint: type fixed, parent world, child room312_two_beams_above_staubli
